File: Desenvolvimento_IC2S-EBM7-2608-V2.3-MOSFET/Projeto_IC2S-EBM7-2608-V2.3-MOSFET/04_barreira.kicad_sch (KiCad schematic)
At the start: 2 parts, among them U5 ISO7141CCDBQR

Commit message: Revisao da reuniao 28-09: ramo unico de 24 V, 100 nF a 50 V, um so MPN de 1 uF
- Saem F2, o diodo e o condensador do ramo +24V_ADC; F1 + diodo alimentam o
  R-78HB e o +24V_ADC. +24V_REG deixa de existir (esquematico, PCB, netclasses).
- Condensador de entrada do R-78HB conferido contra o datasheet Recom (p.4):
  10 uF/100 V cumpre os 3,3 uF/100 V pedidos com Vin > 50 V. Sem alteracao.
- 100 nF fora do 24 V -> TDK C1608X7R1H104K080AA (50 V); o do +24V_ADC fica
  GRM188R72A104KA35D (100 V). 1 uF -> TDK C1608X7R1H105K080AB nos quatro.
- Notas 2, 13 e 14 da folha 2; README e registo em 00-Especificacoes;
  catalogo TDK em Documentos_de_Referencia.

Co-Authored-By: Claude Opus 5.5 (1M context) <noreply@anthropic.com>
Claude-Session: https://claude.ai/code/session_01KPnkiJQKrkjgRqqw9M78ie
Parts:
- C24: value 100nF -> 100nF/50V; MPN GRM188R72A104KA35D -> C1608X7R1H104K080AA
Changed lines of the file:
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@@
 			)
 		)
-		(property "Value" "100nF"
+		(property "Value" "100nF/50V"
 			(at 135.89 62.23 0)
 			(show_name no)
@@
 			)
 		)
-		(property "MPN" "GRM188R72A104KA35D"
+		(property "MPN" "C1608X7R1H104K080AA"
 			(at 6.35 0 0)
 			(hide yes)
