File: Desenvolvimento_IC2S-EBM7-2608-V2.3-MOSFET/Projeto_IC2S-EBM7-2608-V2.3-MOSFET/06_lacos.kicad_sch (KiCad schematic)
At the start: 78 parts, among them Q1 FDN337N, Q2 FDN337N, Q3 FDN337N, Q4 FDN337N, T2 TP_+24V_ADC, U10 TPS26613DDFR, U11 TPS26613DDFR, U12 TPS26613DDFR, U15 TPS7A4001DGN, U9 TPS26613DDFR

Commit message: Revisao da reuniao 28-09: ramo unico de 24 V, 100 nF a 50 V, um so MPN de 1 uF
- Saem F2, o diodo e o condensador do ramo +24V_ADC; F1 + diodo alimentam o
  R-78HB e o +24V_ADC. +24V_REG deixa de existir (esquematico, PCB, netclasses).
- Condensador de entrada do R-78HB conferido contra o datasheet Recom (p.4):
  10 uF/100 V cumpre os 3,3 uF/100 V pedidos com Vin > 50 V. Sem alteracao.
- 100 nF fora do 24 V -> TDK C1608X7R1H104K080AA (50 V); o do +24V_ADC fica
  GRM188R72A104KA35D (100 V). 1 uF -> TDK C1608X7R1H105K080AB nos quatro.
- Notas 2, 13 e 14 da folha 2; README e registo em 00-Especificacoes;
  catalogo TDK em Documentos_de_Referencia.

Co-Authored-By: Claude Opus 5.5 (1M context) <noreply@anthropic.com>
Claude-Session: https://claude.ai/code/session_01KPnkiJQKrkjgRqqw9M78ie
Parts:
- C38, C39, C40, C41, C43, C44, C45, C46, C51: value 100nF -> 100nF/50V; MPN GRM188R72A104KA35D -> C1608X7R1H104K080AA
Changed lines of the file:
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@@
 			)
 		)
-		(property "Value" "100nF"
+		(property "Value" "100nF/50V"
 			(at 78.74 128.27 0)
 			(show_name no)
@@
 			)
 		)
-		(property "MPN" "GRM188R72A104KA35D"
+		(property "MPN" "C1608X7R1H104K080AA"
 			(at 10.16 66.04 0)
 			(hide yes)
@@
 			)
 		)
-		(property "Value" "100nF"
+		(property "Value" "100nF/50V"
 			(at 80.01 200.66 0)
 			(show_name no)
@@
 			)
 		)
-		(property "MPN" "GRM188R72A104KA35D"
+		(property "MPN" "C1608X7R1H104K080AA"
 			(at 11.43 138.43 0)
 			(hide yes)
@@
 			)
 		)
-		(property "Value" "100nF"
+		(property "Value" "100nF/50V"
 			(at 87.63 270.51 0)
 			(show_name no)
@@
 			)
 		)
-		(property "MPN" "GRM188R72A104KA35D"
+		(property "MPN" "C1608X7R1H104K080AA"
 			(at 19.05 208.28 0)
 			(hide yes)
@@
 			)
 		)
-		(property "Value" "100nF"
+		(property "Value" "100nF/50V"
 			(at 78.74 62.23 0)
 			(show_name no)
@@
 			)
 		)
-		(property "MPN" "GRM188R72A104KA35D"
+		(property "MPN" "C1608X7R1H104K080AA"
 			(at 10.16 0 0)
 			(hide yes)
@@
 			)
 		)
-		(property "Value" "100nF"
+		(property "Value" "100nF/50V"
 			(at 95.504 246.38 0)
 			(show_name no)
@@
 			)
 		)
-		(property "MPN" "GRM188R72A104KA35D"
+		(property "MPN" "C1608X7R1H104K080AA"
 			(at 91.44 245.11 0)
 			(hide yes)
@@
 			)
 		)
-		(property "Value" "100nF"
+		(property "Value" "100nF/50V"
 			(at 90.424 109.728 0)
 			(show_name no)
@@
 			)
 		)
-		(property "MPN" "GRM188R72A104KA35D"
+		(property "MPN" "C1608X7R1H104K080AA"
 			(at 87.63 107.95 0)
 			(hide yes)
@@
 			)
 		)
-		(property "Value" "100nF"
+		(property "Value" "100nF/50V"
 			(at 94.742 183.896 0)
 			(show_name no)
@@
 			)
 		)
-		(property "MPN" "GRM188R72A104KA35D"
+		(property "MPN" "C1608X7R1H104K080AA"
 			(at 90.17 182.88 0)
 			(hide yes)
@@
 			)
 		)
-		(property "Value" "100nF"
+		(property "Value" "100nF/50V"
 			(at 246.38 67.31 0)
 			(show_name no)
@@
 			)
 		)
-		(property "MPN" "GRM188R72A104KA35D"
+		(property "MPN" "C1608X7R1H104K080AA"
 			(at 245.11 66.04 0)
 			(hide yes)
@@
 			)
 		)
-		(property "Value" "100nF"
+		(property "Value" "100nF/50V"
 			(at 80.01 39.37 0)
 			(show_name no)
@@
 			)
 		)
-		(property "MPN" "GRM188R72A104KA35D"
+		(property "MPN" "C1608X7R1H104K080AA"
 			(at 78.74 38.1 0)
 			(hide yes)
