File: Desenvolvimento_IC2S-EBM7-2608-V2.3-MOSFET/Projeto_IC2S-EBM7-2608-V2.3-MOSFET/IC2S-EBM7-2608-V2.3-MOSFET.kicad_pcb (KiCad board)
At the start: 4 copper layers, 60 x 60 mm, 168 parts, among them P1 M20-7822046, P2 M20-7821446, Q1 FDN337N, Q2 FDN337N, Q3 FDN337N, Q4 FDN337N, T1 TP_+24V, T10 TP_DGND, T2 TP_+24V_ADC, T4 TP_+5V_REG, T5 TP_+3.3V_ANA, T6 TP_+3.3V_DIG, T7 TP_GND_ADC_P1, T8 TP_GND_ADC, U10 TPS26613DDFR, U11 TPS26613DDFR, U12 TPS26613DDFR, U13 LP5907MFX-2.5, U14 TL431B, U15 TPS7A4001DGN, U3 R-78HB5.0-0.5L, U4 SPX3819M5-L-3-3/TR, U5 ISO7141CCDBQR, U6 AD7124-8BCPZ, U7 ADR4525BRZ, U8 MCP1824ST-3302E/DB, U9 TPS26613DDFR

Commit message: Revisao da reuniao 28-09: ramo unico de 24 V, 100 nF a 50 V, um so MPN de 1 uF
- Saem F2, o diodo e o condensador do ramo +24V_ADC; F1 + diodo alimentam o
  R-78HB e o +24V_ADC. +24V_REG deixa de existir (esquematico, PCB, netclasses).
- Condensador de entrada do R-78HB conferido contra o datasheet Recom (p.4):
  10 uF/100 V cumpre os 3,3 uF/100 V pedidos com Vin > 50 V. Sem alteracao.
- 100 nF fora do 24 V -> TDK C1608X7R1H104K080AA (50 V); o do +24V_ADC fica
  GRM188R72A104KA35D (100 V). 1 uF -> TDK C1608X7R1H105K080AB nos quatro.
- Notas 2, 13 e 14 da folha 2; README e registo em 00-Especificacoes;
  catalogo TDK em Documentos_de_Referencia.

Co-Authored-By: Claude Opus 5.5 (1M context) <noreply@anthropic.com>
Claude-Session: https://claude.ai/code/session_01KPnkiJQKrkjgRqqw9M78ie
Parts:
- removed C1: 10uF/100V, EBM7_V23:C_1210_3225Metric
- removed D1: MBR1H100SF, EBM7_V23:SOD123
- removed F2: CC12H750MA-TR, EBM7_V23:1206F
- C18, C20, C22, C23, C24, C25, C27, C28, C34, C35, C37, C38, C39, C40, C41, C43, C44, C45, C46, C51, C54, C55, C58, C59: value 100nF -> 100nF/50V
- C26, C57: value 1uF -> 1uF/50V
- C52, C53: value 1uF/16V -> 1uF/50V
Connections:
- C13 pad 1: +24V_REG -> +24V_ADC
- D5 pad 1: +24V_REG -> +24V_ADC
- U3 pad 1: +24V_REG -> +24V_ADC
Routing:
- net +24V_REG: track 8.88 -> 0.00 mm
- net +24V_ADC: track 110.6 -> 118.5 mm
- net +24V: track 17.8 -> 14.2 mm
- net Net-(D1-A): track 2.20 -> 0.00 mm
- net GND_ADC: track 150.6 -> 148.6 mm

Commit message: LDO 3,3 V do lado PLC: U8 MCP1824ST (SOT-223) -> SPX3819M5-L-3-3/TR (SOT-23-5), mesmo MPN do U4
- Criterio da equipa: menos MPN, mais pecas do mesmo tipo; o MCP1824ST sai.
- EN a VIN, BYP aberto; estabilidade com ceramico sem garantia no datasheet (provada em campo na V2.2).
- Esquematico: ERC 0; netlist so muda os pinos do U8. PCB: pegada SOT-23-5 no
  mesmo sitio; faltam rotear 6 ligacoes do U8.
- Registo: alteracao_LDO_3V3_lado_PLC_2026-09-28.md (comparacao, verificacao e
  riscos em aberto). BOM e PDF do esquematico regenerados.

Co-Authored-By: Claude Opus 5.5 (1M context) <noreply@anthropic.com>
Claude-Session: https://claude.ai/code/session_01KPnkiJQKrkjgRqqw9M78ie
Parts:
- U8: value MCP1824ST-3302E/DB -> SPX3819M5-L-3-3/TR; footprint EBM7_V23:SOT-223-3 -> EBM7_V23:SOT-23-5
Connections:
- U8 pad 3: +3.3V -> +5V
- U8 pad 4: DGND -> unconnected-(U8-BP-Pad4)
Routing:
- net +5V: track 11.9 -> 6.29 mm
- net +3.3V: track 46.1 -> 42.4 mm
- net DGND: track 9.72 -> 8.02 mm, vias 9 -> 3

Commit message: C61 2,2 uF na saida do U8 (SPX3819), como a saida do SPX da V2.2 em campo
- Mesmo complemento da fixa (datasheet SPX3819 Fig. 18). PCB: clone do C48 a 3 mm do U8.
- ERC 0; DRC 0 erros, sem avisos novos, paridade 1 (C35, anterior).

Co-Authored-By: Claude Opus 5.5 (1M context) <noreply@anthropic.com>
Claude-Session: https://claude.ai/code/session_01KPnkiJQKrkjgRqqw9M78ie
Parts:
- added C61: 2.2uF, EBM7_V23:0603C, F.Cu at (128.2, 111.8)
Changed lines of the file:
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@@
+		)
+	)
+	(footprint "EBM7_V23:0603C"
+		(layer "F.Cu")
+		(at 128.25 111.75)
+		(descr "2Solve PCB Library '0603C', recuperado da PCB V2.2 (fabricada) em 2026-09-04.")
+		(property "Reference" "C61"
+			(at 2.355 -1.57 0)
+			(layer "F.SilkS")
+			(effects
+				(font
+					(size 0.6 0.6)
+					(thickness 0.1)
+				)
+			)
+		)
+		(property "Value" "2.2uF"
+			(at -3.72999 -0.3429 270)
+			(unlocked yes)
+			(layer "F.SilkS")
+			(hide yes)
+			(effects
+				(font
+					(size 1.524 1.524)
+					(thickness 0.254)
+				)
+				(justify left bottom)
+			)
+		)
+		(property "Datasheet" ""
+			(at 0 0 0)
+			(layer "F.Fab")
+			(hide yes)
+			(effects
+				(font
+					(size 1.27 1.27)
+				)
+			)
+		)
+		(property "Description" ""
+			(at 0 0 0)
+			(layer "F.Fab")
+			(hide yes)
+			(effects
+				(font
+					(size 1.27 1.27)
+				)
+			)
+		)
+		(property "MPN" "C1608X5R1E225K080AB"
+			(at 0 0 0)
+			(unlocked yes)
+			(layer "F.Fab")
+			(hide yes)
+			(effects
+				(font
+					(size 1 1)
+					(thickness 0.15)
+				)
+			)
+		)
+		(property ki_fp_filters "C_*")
+		(sheetname "/3 Alimentacao/")
+		(sheetfile "03_alimentacao.kicad_sch")
+		(attr smd)
+		(duplicate_pad_numbers_are_jumpers no)
+		(fp_line
+			(start -0.1 -0.45)
+			(end 0.1 -0.45)
+			(stroke
+				(width 0.1)
+				(type solid)
+			)
+			(layer "F.SilkS")
+		)
+		(fp_line
+			(start -0.1 0.45)
+			(end 0.1 0.45)
+			(stroke
+				(width 0.1)
+				(type solid)
+			)
+			(layer "F.SilkS")
+		)
+		(fp_rect
+			(start -1.35 -0.7)
+			(end 1.35 0.7)
+			(stroke
+				(width 0.05)
+				(type default)
+			)
+			(fill no)
+			(layer "F.CrtYd")
+		)
+		(fp_line
+			(start -0.875 -0.475)
+			(end 0.875 -0.475)
+			(stroke
+				(width 0.1)
+				(type solid)
+			)
+			(layer "User.13")
+		)
+		(fp_line
+			(start -0.875 0.475)
+			(end -0.875 -0.475)
+			(stroke
+				(width 0.1)
+				(type solid)
+			)
+			(layer "User.13")
+		)
+		(fp_line
+			(start -0.875 0.475)
+			(end 0.875 0.475)
+			(stroke
+				(width 0.1)
+				(type solid)
+			)
+			(layer "User.13")
+		)
+		(fp_line
+			(start 0.875 0.475)
+			(end 0.875 -0.475)
+			(stroke
+				(width 0.1)
+				(type solid)
+			)
+			(layer "User.13")
+		)
+		(fp_line
+			(start -1.2 -0.55)
+			(end 1.2 -0.55)
+			(stroke
+				(width 0.1)
+				(type solid)
+			)
+			(layer "User.15")
+		)
+		(fp_line
+			(start -1.2 0.55)
+			(end -1.2 -0.55)
+			(stroke
+				(width 0.1)
+				(type solid)
+			)
+			(layer "User.15")
+		)
+		(fp_line
+			(start -1.2 0.55)
+			(end 1.2 0.55)
+			(stroke
+				(width 0.1)
+				(type solid)
+			)
+			(layer "User.15")
+		)
+		(fp_line
+			(start -0.475 0)
+			(end 0.475 0)
+			(stroke
+				(width 0.1)
+				(type solid)
+			)
+			(layer "User.15")
+		)
+		(fp_line
+			(start 0 0.475)
+			(end 0 -0.475)
+			(stroke
+				(width 0.1)
+				(type solid)
+			)
+			(layer "User.15")
+		)
+		(fp_line
+			(start 1.2 0.55)
+			(end 1.2 -0.55)
+			(stroke
+				(width 0.1)
+				(type solid)
+			)
+			(layer "User.15")
+		)
+		(pad "1" smd rect
+			(at -0.7 0 90)
+			(size 0.9 0.8)
+			(layers "F.Cu" "F.Mask" "F.Paste")
+			(net "DGND")
+			(pintype "passive")
+		)
+		(pad "2" smd rect
+			(at 0.7 0 90)
+			(size 0.9 0.8)
+			(layers "F.Cu" "F.Mask" "F.Paste")
+			(net "+3.3V")
+			(pintype "passive")
+		)
+		(embedded_fonts no)
+		(embedded_files
+			(file
+				(name "User Library-CAPC1608X___CAPC1608X55N.STEP")
+				(type other)
+				(checksum "597E9624E6E4306F77CAACCCC75E6675")
+			)
+		)
+		(model "kicad-embed://User Library-CAPC1608X___CAPC1608X55N.STEP"
+			(offset
+				(xyz 0.00015 0.00016 -0.025)
+			)
+			(scale
+				(xyz 1 1 1)
+			)
+			(rotate
+				(xyz -0 0 0)
+			)
 		)
 	)
